File: pcb/zedekiel/zedekiel.kicad_pcb (KiCad board)
At the start: 2 copper layers, 177 parts, among them K1 KEYSW, K10 KEYSW, K11 KEYSW, K12 KEYSW, K13 KEYSW, K14 KEYSW, K15 KEYSW, K16 KEYSW, K17 KEYSW, K18 KEYSW, K19 KEYSW, K2 KEYSW, K20 KEYSW, K21 KEYSW, K22 KEYSW, K23 KEYSW, K24 KEYSW, K25 KEYSW, K26 KEYSW, K27 KEYSW, K28 KEYSW, K29 KEYSW, K3 KEYSW, K30 KEYSW, K31 KEYSW, K32 KEYSW, K33 KEYSW, K34 KEYSW, K35 KEYSW, K36 KEYSW, K37 KEYSW, K38 KEYSW, K39 KEYSW, K4 KEYSW, K40 KEYSW, K41 KEYSW, K42 KEYSW, K43 KEYSW, K44 KEYSW, K45 KEYSW, K46 KEYSW, K47 KEYSW, K48 KEYSW, K49 KEYSW, K5 KEYSW, K50 KEYSW, K51 KEYSW, K52 KEYSW, K53 KEYSW, K54 KEYSW, K55 KEYSW, K56 KEYSW, K57 KEYSW, K58 KEYSW, K59 KEYSW, K6 KEYSW, K60 KEYSW, K61 KEYSW, K62 KEYSW, K63 KEYSW, K64 KEYSW, K65 KEYSW, K66 KEYSW, K7 KEYSW, K8 KEYSW, K9 KEYSW, SW1 SW_PUSH, U1 ATmega16U4-AU_(modified), X1 16MHz

Commit message: better routing for the switch matrix
Routing:
- net /C14: track 88.1 -> 354.7 mm, vias 0 -> 1
- net /C13: track 90.5 -> 329.0 mm, vias 0 -> 1
- net /C12: track 93.2 -> 304.1 mm, vias 0 -> 1
- net /C11: track 87.8 -> 268.8 mm, vias 0 -> 1
- net /C10: track 89.9 -> 247.6 mm, vias 0 -> 1
- net /C9: track 68.3 -> 214.4 mm, vias 0 -> 1
- net /C8: track 92.2 -> 217.8 mm, vias 0 -> 1
- net /C7: track 88.0 -> 194.8 mm, vias 0 -> 1
- net /C6: track 68.0 -> 155.7 mm, vias 0 -> 1
- net /C5: track 88.3 -> 157.8 mm, vias 0 -> 1
- net /C4: track 87.9 -> 138.0 mm, vias 0 -> 1
- net Net-(R5-Pad1): track 0.00 -> 50.1 mm
- net /C3: track 67.8 -> 101.1 mm, vias 0 -> 1
- net /R5: track 363.3 -> 345.5 mm
- net /C2: track 91.2 -> 106.1 mm, vias 0 -> 1
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Other:
- net class Default: clearance 0.2 -> 0.3
- net class EasyEDA: clearance 0.3 -> 0.2
- net class Power added: clearance 0.2, trace_width 0.3, via_dia 0.8, via_drill 0.4
- rule trace_clearance: 0.2 -> 0.3

Commit message: more routing
Parts:
- moved C5 16.0 mm to (46.8, 109.3), turned to 225 degrees
- moved R6 9.70 mm to (43.3, 112.8), turned to 45 degrees
- moved TP6 0.50 mm to (22.9, 68.9)
- moved TP6 0.50 mm to (22.9, 71.4)
- moved TP5 0.25 mm to (22.9, 76.4)
- moved TP6 0.25 mm to (22.9, 73.9)
- moved TP7 0.25 mm to (22.9, 78.9)
Connections:
- net Net-(R4-Pad1) renamed /D+
- net Net-(R5-Pad1) renamed /D-
Routing:
- net /D+: track 5.56 -> 52.5 mm, vias 0 -> 2
- net /R3: track 278.7 -> 323.6 mm, vias 14 -> 15
- net /C1: track 63.8 -> 101.4 mm, vias 0 -> 2
- net /R4: track 286.5 -> 313.0 mm, vias 14 -> 18
- net /R5: track 345.5 -> 368.5 mm, vias 10 -> 12
- net Net-(C2-Pad1): track 7.64 -> 3.07 mm
- net VCC: track 149.0 -> 153.3 mm, vias 3 -> 2
- net Net-(R6-Pad1): track 0.00 -> 4.23 mm
- net /D-: track 50.1 -> 52.1 mm, vias 0 -> 2
- net /R1: track 350.4 -> 351.3 mm, vias 16 -> 15
- net MISO: track 26.4 -> 25.8 mm
- net /R2: track 343.7 -> 344.2 mm

Commit message: routing improvements
Parts:
- removed the TP6 at (22.9, 68.9)
- removed the TP6 at (22.9, 71.4)
- added TP6: TestPoint, custom:single-pad, B.Cu at (22.9, 76.4)
- added TP6: TestPoint, custom:single-pad, B.Cu at (22.9, 78.9)
- moved TP7 42.4 mm to (53.0, 108.8)
- moved TP5 42.4 mm to (53.0, 106.2)
- moved TP6 42.3 mm to (53.0, 103.6)
- moved C6 0.05 mm to (32.6, 95.8)
Routing:
- net ADC11: track 0.00 -> 13.2 mm
- net SCL: track 0.00 -> 12.4 mm
- net SDA: track 0.00 -> 12.1 mm
- net /R5: track 368.5 -> 366.6 mm, vias 12 -> 11
- net VCC: track 153.3 -> 154.8 mm, vias 2 -> 3
- net /R4: track 313.0 -> 313.9 mm, vias 18 -> 19
- net /C1: track 101.4 -> 101.7 mm, vias 2 -> 4

Commit message: almost done with routing
Routing:
- net /C3: track 101.1 -> 136.6 mm, vias 1 -> 2
- net /C2: track 106.1 -> 141.0 mm, vias 1 -> 2
- net /C4: track 138.0 -> 172.3 mm, vias 1 -> 2
- net /D-: track 52.1 -> 84.9 mm, vias 2 -> 4
- net /D+: track 52.5 -> 84.3 mm, vias 2 -> 4
- net /C5: track 157.8 -> 188.1 mm, vias 1 -> 2
- net /C6: track 155.7 -> 184.7 mm, vias 1 -> 2
- net /C8: track 217.8 -> 245.4 mm, vias 1 -> 2
- net /C14: track 354.7 -> 379.4 mm, vias 1 -> 4
- net /C7: track 194.8 -> 218.1 mm, vias 1 -> 2
- net /C11: track 268.8 -> 289.0 mm, vias 1 -> 2
- net /C13: track 329.0 -> 348.4 mm, vias 1 -> 2
- net /C12: track 304.1 -> 323.2 mm, vias 1 -> 2
- net /C10: track 247.6 -> 260.8 mm, vias 1 -> 2
- net /C9: track 214.4 -> 226.2 mm, vias 1 -> 2
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
Commit message: basically done with routing
Parts:
- moved C2 0.81 mm to (27.8, 108.8)
- moved C3 0.81 mm to (24.4, 108.8), turned to 180 degrees
- moved C1 0.81 mm to (24.4, 107.2), turned to 180 degrees
- moved X1 0.81 mm to (26.1, 111.6)
Routing:
- net Net-(R1-Pad2): track 3.05 -> 28.2 mm, vias 1 -> 3
- net Net-(C3-Pad1): track 3.07 -> 24.3 mm, vias 0 -> 2
- net Net-(C2-Pad1): track 3.07 -> 21.1 mm, vias 0 -> 2
- net VCC: track 154.6 -> 158.8 mm
- net Net-(C1-Pad1): track 16.0 -> 13.2 mm
- net /C2: track 141.0 -> 142.4 mm
- net /R5: track 367.9 -> 367.0 mm
- net /C10: track 260.8 -> 260.0 mm

Commit message: done with routing
Routing:
- net VCC: track 158.8 -> 0.63 mm, vias 3 -> 0
- net Net-(R1-Pad2): track 28.2 -> 24.2 mm
- net GND: track 0.03 -> 1.63 mm, vias 45 -> 24
- net (no net): vias 20 -> 0
- added copper zone on F.Cu, net GND
- added copper zone on B.Cu, net VCC
Other:
- board outline added: 304 x 95 mm

Commit message: labeling & silk screen art
Parts:
- added G***: LOGO, custom:silkscreen-art, F.Cu at (172.9, 68.3)
Routing:
- net /C2: track 142.4 -> 144.8 mm
- net GND: track 1.63 -> 3.15 mm
- net /R1: track 351.8 -> 351.0 mm
Other:
- board text added: "ADC"
- board text added: "GND"
- board text added: "MISO"
- board text added: "MOSI"
- board text added: "SCL"
- board text added: "SCLK"
- board text added: "SDA"
- board text added: "VCC"

Commit message: signarue
Parts:
- added G***: LOGO, custom:signature, B.Cu at (313.4, 112.9)
Changed lines of the file:
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@@
     (tracks 1130)
     (zones 0)
-    (modules 178)
+    (modules 179)
     (nets 113)
   )
@@
     (add_net VCC)
   )
+  (module custom:signature (layer B.Cu)
+    (at 313.4 112.9 180)
+    (fp_text reference G*** (at 0 0) (layer B.SilkS) hide
+      (effects (font (size 1.524 1.524) (thickness 0.3)) (justify mirror))
+    )
+    (fp_text value LOGO (at 0.75 0) (layer B.SilkS) hide
+      (effects (font (size 1.524 1.524) (thickness 0.3)) (justify mirror))
+    )
+    (fp_poly (pts (xy -0.154198 1.142898) (xy -0.09976 1.092378) (xy -0.028656 1.025474) (xy 0.04531 0.955187)
+      (xy 0.058208 0.942849) (xy 0.1905 0.816139) (xy 0.1905 0.559602) (xy 0.191542 0.438273)
+      (xy 0.194388 0.292198) (xy 0.198615 0.138903) (xy 0.203804 -0.004084) (xy 0.204388 -0.017801)
+      (xy 0.218276 -0.338667) (xy 0.290159 -0.338667) (xy 0.32844 -0.343268) (xy 0.368201 -0.360524)
+      (xy 0.417371 -0.395611) (xy 0.483883 -0.453705) (xy 0.524979 -0.491923) (xy 0.592799 -0.556558)
+      (xy 0.648225 -0.610975) (xy 0.684469 -0.648411) (xy 0.694972 -0.661256) (xy 0.678076 -0.667546)
+      (xy 0.626861 -0.672683) (xy 0.549333 -0.676125) (xy 0.456847 -0.677334) (xy 0.352014 -0.677654)
+      (xy 0.282338 -0.679544) (xy 0.240641 -0.684399) (xy 0.219746 -0.693612) (xy 0.212476 -0.708576)
+      (xy 0.211648 -0.724959) (xy 0.195621 -0.764114) (xy 0.148057 -0.829704) (xy 0.069698 -0.920776)
+      (xy 0.001042 -0.994834) (xy -0.209546 -1.217084) (xy -0.210607 -0.936625) (xy -0.211667 -0.656167)
+      (xy -0.287989 -0.656167) (xy -0.327544 -0.652225) (xy -0.366618 -0.636894) (xy -0.413526 -0.60491)
+      (xy -0.476587 -0.551014) (xy -0.526114 -0.505524) (xy -0.59399 -0.441131) (xy -0.649405 -0.386298)
+      (xy -0.685441 -0.348007) (xy -0.695498 -0.334614) (xy -0.67899 -0.326072) (xy -0.624918 -0.321062)
+      (xy -0.537927 -0.319855) (xy -0.466745 -0.321215) (xy -0.230409 -0.328084) (xy -0.232361 0.444077)
+      (xy -0.234312 1.216237) (xy -0.154198 1.142898)) (layer B.SilkS) (width 0.01))
+    (fp_poly (pts (xy -5.127388 0.155505) (xy -5.132917 -0.704989) (xy -5.3975 -0.901554) (xy -5.489771 -0.969163)
+      (xy -5.570817 -1.02678) (xy -5.634302 -1.070038) (xy -5.673892 -1.094571) (xy -5.68325 -1.098502)
+      (xy -5.706657 -1.086036) (xy -5.756167 -1.051579) (xy -5.825154 -0.99999) (xy -5.906991 -0.936126)
+      (xy -5.931959 -0.916182) (xy -6.1595 -0.733478) (xy -6.1595 -0.315912) (xy -5.963709 -0.321998)
+      (xy -5.767917 -0.328084) (xy -5.761352 -0.39597) (xy -5.747113 -0.445993) (xy -5.709752 -0.496671)
+      (xy -5.650227 -0.5514) (xy -5.545667 -0.638942) (xy -5.545667 1.016) (xy -5.121859 1.016)
+      (xy -5.127388 0.155505)) (layer B.SilkS) (width 0.01))
+    (fp_poly (pts (xy -3.994213 0.935732) (xy -3.915834 0.855465) (xy -3.915834 -0.69504) (xy -4.190822 -0.897853)
+      (xy -4.284597 -0.966311) (xy -4.366658 -1.024889) (xy -4.430923 -1.06935) (xy -4.471308 -1.095455)
+      (xy -4.481864 -1.100574) (xy -4.503398 -1.088011) (xy -4.551324 -1.053618) (xy -4.619158 -1.002236)
+      (xy -4.700415 -0.938703) (xy -4.725459 -0.918781) (xy -4.953 -0.737081) (xy -4.953 -0.440578)
+      (xy -4.572731 -0.440578) (xy -4.461605 -0.537789) (xy -4.405836 -0.585921) (xy -4.36413 -0.620686)
+      (xy -4.345057 -0.634952) (xy -4.344822 -0.635) (xy -4.343395 -0.614702) (xy -4.342101 -0.557284)
+      (xy -4.340985 -0.467958) (xy -4.340096 -0.351938) (xy -4.339481 -0.214435) (xy -4.339186 -0.060664)
+      (xy -4.339167 -0.009477) (xy -4.339167 0.616045) (xy -4.450292 0.609648) (xy -4.561417 0.60325)
+      (xy -4.572731 -0.440578) (xy -4.953 -0.440578) (xy -4.953 0.849514) (xy -4.884209 0.932375)
+      (xy -4.815417 1.015237) (xy -4.444005 1.015618) (xy -4.072592 1.016) (xy -3.994213 0.935732)) (layer B.SilkS) (width 0.01))
+    (fp_poly (pts (xy 2.495888 0.933579) (xy 2.528687 0.888905) (xy 2.548176 0.848506) (xy 2.557783 0.799039)
+      (xy 2.560937 0.727159) (xy 2.561166 0.679579) (xy 2.561166 0.508) (xy 2.137833 0.508)
+      (xy 2.137833 0.637212) (xy 1.915583 0.624416) (xy 1.909484 0.46502) (xy 1.903386 0.305624)
+      (xy 2.226984 0.133607) (xy 2.550583 -0.03841) (xy 2.562157 -0.733582) (xy 2.286629 -0.917125)
+      (xy 2.191249 -0.979952) (xy 2.108093 -1.033387) (xy 2.043553 -1.073428) (xy 2.004019 -1.096073)
+      (xy 1.995092 -1.099661) (xy 1.973514 -1.086817) (xy 1.925464 -1.052294) (xy 1.857457 -1.000946)
+      (xy 1.77601 -0.937624) (xy 1.751541 -0.918297) (xy 1.524 -0.737938) (xy 1.524 -0.381)
+      (xy 1.712031 -0.381) (xy 1.803419 -0.382063) (xy 1.860843 -0.38631) (xy 1.892644 -0.395329)
+      (xy 1.907162 -0.41071) (xy 1.909917 -0.418686) (xy 1.930533 -0.451053) (xy 1.974738 -0.498682)
+      (xy 2.028802 -0.547657) (xy 2.137833 -0.638942) (xy 2.137833 -0.241579) (xy 1.830916 -0.066391)
+      (xy 1.524 0.108796) (xy 1.524 0.492296) (xy 1.52428 0.629444) (xy 1.525602 0.731127)
+      (xy 1.528687 0.80421) (xy 1.534256 0.855561) (xy 1.54303 0.892046) (xy 1.555731 0.920531)
+      (xy 1.571625 0.945754) (xy 1.61925 1.015711) (xy 2.024929 1.015855) (xy 2.430609 1.016)
+      (xy 2.495888 0.933579)) (layer B.SilkS) (width 0.01))
+    (fp_poly (pts (xy 3.725333 -0.461725) (xy 3.831166 -0.550334) (xy 3.937 -0.638942) (xy 3.937 -0.275167)
+      (xy 4.361814 -0.275167) (xy 4.34975 -0.705101) (xy 4.085166 -0.90161) (xy 3.992891 -0.969203)
+      (xy 3.911843 -1.026806) (xy 3.848357 -1.070052) (xy 3.80877 -1.094575) (xy 3.799416 -1.098502)
+      (xy 3.77601 -1.086036) (xy 3.726499 -1.051579) (xy 3.657512 -0.99999) (xy 3.575676 -0.936126)
+      (xy 3.550708 -0.916182) (xy 3.323166 -0.733478) (xy 3.323166 1.016) (xy 3.725333 1.016)
+      (xy 3.725333 -0.461725)) (layer B.SilkS) (width 0.01))
+    (fp_poly (pts (xy 4.931833 -0.461725) (xy 5.037666 -0.550334) (xy 5.1435 -0.638942) (xy 5.1435 -0.275167)
+      (xy 5.568314 -0.275167) (xy 5.55625 -0.705101) (xy 5.291666 -0.90161) (xy 5.199391 -0.969203)
+      (xy 5.118343 -1.026806) (xy 5.054857 -1.070052) (xy 5.01527 -1.094575) (xy 5.005916 -1.098502)
+      (xy 4.98251 -1.086036) (xy 4.932999 -1.051579) (xy 4.864012 -0.99999) (xy 4.782176 -0.936126)
+      (xy 4.757208 -0.916182) (xy 4.529666 -0.733478) (xy 4.529666 1.016) (xy 4.931833 1.016)
+      (xy 4.931833 -0.461725)) (layer B.SilkS) (width 0.01))
+    (fp_poly (pts (xy -3.220769 0.703791) (xy -3.114843 0.391583) (xy -3.113172 0.703791) (xy -3.1115 1.016)
+      (xy -2.709334 1.016) (xy -2.709334 -0.740512) (xy -2.89136 -0.883548) (xy -2.966448 -0.942043)
+      (xy -3.029302 -0.990053) (xy -3.072485 -1.021958) (xy -3.087968 -1.032148) (xy -3.098372 -1.01475)
+      (xy -3.118223 -0.963039) (xy -3.145332 -0.883405) (xy -3.177511 -0.782236) (xy -3.207568 -0.682898)
+      (xy -3.312584 -0.328084) (xy -3.318387 -0.682625) (xy -3.321171 -0.799661) (xy -3.32522 -0.900246)
+      (xy -3.330123 -0.977492) (xy -3.335467 -1.02451) (xy -3.339554 -1.035791) (xy -3.36151 -1.023111)
+      (xy -3.409677 -0.989677) (xy -3.476805 -0.940665) (xy -3.550709 -0.88502) (xy -3.7465 -0.735626)
+      (xy -3.7465 1.016) (xy -3.326695 1.016) (xy -3.220769 0.703791)) (layer B.SilkS) (width 0.01))
+    (fp_poly (pts (xy -2.014269 0.703791) (xy -1.908343 0.391583) (xy -1.906672 0.703791) (xy -1.905 1.016)
+      (xy -1.502834 1.016) (xy -1.502834 -0.740512) (xy -1.68486 -0.883548) (xy -1.759948 -0.942043)
+      (xy -1.822802 -0.990053) (xy -1.865985 -1.021958) (xy -1.881468 -1.032148) (xy -1.891872 -1.01475)
+      (xy -1.911723 -0.963039) (xy -1.938832 -0.883405) (xy -1.971011 -0.782236) (xy -2.001068 -0.682898)
+      (xy -2.106084 -0.328084) (xy -2.111887 -0.682625) (xy -2.114671 -0.799661) (xy -2.11872 -0.900246)
+      (xy -2.123623 -0.977492) (xy -2.128967 -1.02451) (xy -2.133054 -1.035791) (xy -2.15501 -1.023111)
+      (xy -2.203177 -0.989677) (xy -2.270305 -0.940665) (xy -2.344209 -0.88502) (xy -2.54 -0.735626)
+      (xy -2.54 1.016) (xy -2.120195 1.016) (xy -2.014269 0.703791)) (layer B.SilkS) (width 0.01))
+    (fp_poly (pts (xy 3.153833 -0.694497) (xy 2.968625 -0.829734) (xy 2.89028 -0.886662) (xy 2.823049 -0.935)
+      (xy 2.775251 -0.9688) (xy 2.756958 -0.981151) (xy 2.750638 -0.977179) (xy 2.745347 -0.954915)
+      (xy 2.741005 -0.911427) (xy 2.737534 -0.84378) (xy 2.734856 -0.74904) (xy 2.732893 -0.624273)
+      (xy 2.731566 -0.466546) (xy 2.730797 -0.272923) (xy 2.730507 -0.040472) (xy 2.7305 0.009334)
+      (xy 2.7305 1.016) (xy 3.153833 1.016) (xy 3.153833 -0.694497)) (layer B.SilkS) (width 0.01))
+    (fp_poly (pts (xy -5.122334 1.100666) (xy -5.545667 1.100666) (xy -5.545667 1.4605) (xy -5.122334 1.4605)
+      (xy -5.122334 1.100666)) (layer B.SilkS) (width 0.01))
+    (fp_poly (pts (xy 3.153833 1.100666) (xy 2.7305 1.100666) (xy 2.7305 1.4605) (xy 3.153833 1.4605)
+      (xy 3.153833 1.100666)) (layer B.SilkS) (width 0.01))
+  )
   (module custom:silkscreen-art (layer F.Cu)
