File: pcb/zedekiel.kicad_pcb (KiCad board)
At the start: 2 copper layers, 304 x 95 mm, 179 parts, among them K1 KEYSW, K10 KEYSW, K11 KEYSW, K12 KEYSW, K13 KEYSW, K14 KEYSW, K15 KEYSW, K16 KEYSW, K17 KEYSW, K18 KEYSW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

Commit message: added a librecad scketch of the pcb
Parts:
- moved USB1 0.20 mm to (47.6, 19.4)
Routing:
- net Net-(R5-Pad2): track 23.2 -> 21.9 mm
