File: pcb/zedekiel.kicad_pcb (KiCad board)
At the start: 2 copper layers, 304 x 95 mm, 179 parts, among them K1 KEYSW, K10 KEYSW, K11 KEYSW, K12 KEYSW, K13 KEYSW, K14 KEYSW, K15 KEYSW, K16 KEYSW, K17 KEYSW, K18 KEYSW, K19 KEYSW, K2 KEYSW, K20 KEYSW, K21 KEYSW, K22 KEYSW, K23 KEYSW, K24 KEYSW, K25 KEYSW, K26 KEYSW, K27 KEYSW, K28 KEYSW, K29 KEYSW, K3 KEYSW, K30 KEYSW, K31 KEYSW, K32 KEYSW, K33 KEYSW, K34 KEYSW, K35 KEYSW, K36 KEYSW, K37 KEYSW, K38 KEYSW, K39 KEYSW, K4 KEYSW, K40 KEYSW, K41 KEYSW, K42 KEYSW, K43 KEYSW, K44 KEYSW, K45 KEYSW, K46 KEYSW, K47 KEYSW, K48 KEYSW, K49 KEYSW, K5 KEYSW, K50 KEYSW, K51 KEYSW, K52 KEYSW, K53 KEYSW, K54 KEYSW, K55 KEYSW, K56 KEYSW, K57 KEYSW, K58 KEYSW, K59 KEYSW, K6 KEYSW, K60 KEYSW, K61 KEYSW, K62 KEYSW, K63 KEYSW, K64 KEYSW, K65 KEYSW, K66 KEYSW, K7 KEYSW, K8 KEYSW, K9 KEYSW, SW1 SW_PUSH, U1 ATmega16U4-AU_(modified), X1 16MHz

Commit message: proper passhthough holes, better hole indicators, updated 3d model paths, freecad export of pcb
Parts:
- removed the REF** at (47.4, 88.8)
- removed the REF** at (248.4, 65.5)
- removed the REF** at (115.4, 65.5)
- removed the REF** at (46.0, 39.4)
- removed the REF** at (298.9, 35.4)
- removed the REF** at (162.9, 38.8)
- removed the REF** at (297.0, 95.0)
- removed the REF** at (166.4, 105.9)
- added REF**: MountingHole_4.5mm, custom:MountingHole_with_indicator_4.5mm, F.Cu at (297.0, 95.0)
- added REF**: MountingHole_4.5mm, custom:MountingHole_with_indicator_4.5mm, F.Cu at (166.4, 105.9)
- added REF**: MountingHole_4.5mm, custom:MountingHole_with_indicator_4.5mm, F.Cu at (248.4, 65.5)
- added REF**: MountingHole_4.5mm, custom:MountingHole_with_indicator_4.5mm, F.Cu at (115.4, 65.5)
- added REF**: MountingHole_4.5mm, custom:MountingHole_with_indicator_4.5mm, F.Cu at (47.4, 88.8)
- added REF**: MountingHole_4.5mm, custom:MountingHole_with_indicator_4.5mm, F.Cu at (298.9, 35.4)
- added REF**: MountingHole_4.5mm, custom:MountingHole_with_indicator_4.5mm, F.Cu at (162.9, 38.8)
- added REF**: MountingHole_4.5mm, custom:MountingHole_with_indicator_4.5mm, F.Cu at (46.0, 39.4)
Routing:
- net GND: vias 24 -> 16

Commit message: designing the new case
Parts:
- K1, K43, K56, K66: footprint custom:Kailh_socket_MX_1.50U -> custom:Kailh_socket_MX_with_switch_1.50U
- K10, K11, K12, K13, K14, K16, K17, K18, K19, K2, K20, K21, K22, K23, K24, K25, K26, K27, K3, K30, K31, K32, K33, K34, K35, K36, K37, K38, K39, K4, K40, K41, K44, K45, K46, K47, K48, K49, K5, K50, K51, K52, K53, K54, K59, K6, K7, K8, K9: footprint custom:Kailh_socket_MX_1.00U -> custom:Kailh_socket_MX_with_switch_1.50U
- K15: footprint custom:Kailh_socket_MX_1.75U -> custom:Kailh_socket_MX_with_switch_1.50U
- K28, K60: footprint custom:Kailh_socket_MX_2.25U -> custom:Kailh_socket_MX_with_switch_1.50U
- K29, K42, K55, K57, K64: footprint custom:Kailh_socket_MX_2.00U -> custom:Kailh_socket_MX_with_switch_1.50U
- K58, K61, K62, K63, K65: footprint custom:Kailh_socket_MX_1.25U -> custom:Kailh_socket_MX_with_switch_1.50U

Commit message: low case finished, test assembly
Parts:
- K1, K10, K11, K12, K13, K14, K15, K16, K17, K18, K19, K2, K20, K21, K22, K23, K24, K25, K26, K27, K28, K29, K3, K30, K31, K32, K33, K34, K35, K36, K37, K38, K39, K4, K40, K41, K42, K43, K44, K45, K46, K47, K48, K49, K5, K50, K51, K52, K53, K54, K55, K56, K57, K58, K59, K6, K60, K61, K62, K63, K64, K65, K66, K7, K8, K9: footprint custom:Kailh_socket_MX_with_switch_1.50U -> custom:Kailh_socket_MX_with_switch_1.00U
