File: zedekiel/zedekiel.kicad_pcb (KiCad board)
At the start: 2 copper layers, 304 x 95 mm, 181 parts, among them K1 KEYSW, K10 KEYSW, K11 KEYSW, K12 KEYSW, K13 KEYSW, K14 KEYSW, K15 KEYSW, K16 KEYSW, K17 KEYSW, K18 KEYSW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

Commit message: Fixed a problem on the pcb, updated readme
Parts:
- renumbered TP3 to TP2, TP2 to TP3
Connections:
- TP2 pad 1: Net-(R5-Pad2) -> Net-(R4-Pad2)
- TP3 pad 1: Net-(R4-Pad2) -> Net-(R5-Pad2)
Routing:
- net Net-(R4-Pad2): track 17.4 -> 21.6 mm, vias 2 -> 0
- net Net-(R5-Pad2): track 22.0 -> 17.9 mm, vias 0 -> 2
